File: interface/schematic.brd (EAGLE design)
At the start: 100 x 46 mm, 31 parts, among them J1 AUDIO_JACK_3.5MM_KIT, J2 AUDIO_JACK_3.5MM_KIT, J3 RJ45, T1 2N3904, T2 2N3904

Commit message: Added decals
Parts:
- R11: value 4K7 -> 3K3
Other:
- board text added: "https://github.com/ivica3730k/AFSK-Ham-Radio-Interface"
- board text added: "https://ivica-matic.com"
Changed lines of the file:
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@@
 <layer number="26" name="bNames" color="7" fill="1" visible="yes" active="yes"/>
 <layer number="27" name="tValues" color="7" fill="1" visible="yes" active="yes"/>
-<layer number="28" name="bValues" color="7" fill="1" visible="no" active="yes"/>
+<layer number="28" name="bValues" color="7" fill="1" visible="yes" active="yes"/>
 <layer number="29" name="tStop" color="7" fill="3" visible="no" active="yes"/>
 <layer number="30" name="bStop" color="7" fill="6" visible="no" active="yes"/>
@@
 <hole x="23" y="43" drill="1"/>
 <hole x="23" y="45" drill="1"/>
+<text x="83" y="6" size="1.27" layer="28" rot="MR90">https://github.com/ivica3730k/AFSK-Ham-Radio-Interface</text>
+<text x="85" y="6" size="1.27" layer="28" rot="MR90">https://ivica-matic.com</text>
 </plain>
 <attributes>
@@
 <attribute name="VALUE" x="75.7434" y="21.4894" size="0.508" layer="27" ratio="10" rot="R90"/>
 </element>
-<element name="R11" library="rcl" library_urn="urn:adsk.eagle:library:334" package="0207/10" package3d_urn="urn:adsk.eagle:package:23491/2" value="4K7" x="64.25" y="8.5" smashed="yes">
+<element name="R11" library="rcl" library_urn="urn:adsk.eagle:library:334" package="0207/10" package3d_urn="urn:adsk.eagle:package:23491/2" value="3K3" x="64.25" y="8.5" smashed="yes">
 <attribute name="NAME" x="61.202" y="10.024" size="1.27" layer="25" ratio="10"/>
 <attribute name="POPULARITY" value="81" x="64.25" y="8.5" size="0.8128" layer="27" display="off"/>
